Commit message: Added Camera sensor

File: urdf/roomba/slambot.gazebo.xacro (robot description, xacro)
@@ -50,14 +50,17 @@
         <slip2 value = "1.0"/>
     </gazebo>
-<!--Camera Plugin
-    <gazebo reference="camera">
+<!--Camera Plugin-->
+  <gazebo reference="camera">
     <material>Gazebo/Red</material>
     <sensor type="camera" name="camera1">
+      <pose>0.2 0 0.055 0 0 0</pose>
+      <visualize>true</visualize>
       <update_rate>30.0</update_rate>
+      <always_on>true</always_on>
       <camera name="head">
-        <horizontal_fov>1.3962634</horizontal_fov>
+        <horizontal_fov>1.089</horizontal_fov>
         <image>
-          <width>800</width>
-          <height>800</height>
+          <width>640</width>
+          <height>480</height>
           <format>R8G8B8</format>
         </image>
@@ -68,20 +71,10 @@
       </camera>
       <plugin name="camera_controller" filename="libgazebo_ros_camera.so">
-        <alwaysOn>true</alwaysOn>
-        <updateRate>0.0</updateRate>
-        <cameraName>mybot/camera1</cameraName>
-        <imageTopicName>image_raw</imageTopicName>
-        <cameraInfoTopicName>camera_info</cameraInfoTopicName>
-        <frameName>camera</frameName>
-        <hackBaseline>0.07</hackBaseline>
-        <distortionK1>0.0</distortionK1>
-        <distortionK2>0.0</distortionK2>
-        <distortionK3>0.0</distortionK3>
-        <distortionT1>0.0</distortionT1>
-        <distortionT2>0.0</distortionT2>
+        <camera_name>slambot/camera1</camera_name>
+        <frame_name>camera</frame_name>
+        <hack_baseline>0.07</hack_baseline>
       </plugin>
     </sensor>
   </gazebo>
--->
 <!-- hokuyo -->
   <gazebo reference="hokuyo">
@@ -116,5 +109,5 @@
       <plugin name="gazebo_ros_head_hokuyo_controller" filename="libgazebo_ros_ray_sensor.so">
         <ros>
-          <namespace>/slambot/laser</namespace>
+          <namespace>/</namespace>
           <remapping>~/out:=scan</remapping>
         </ros>

File: urdf/roomba/slambot.xacro (robot description, xacro)
@@ -120,5 +120,5 @@
     <joint_properties damping="1" friction="0"/>
   </joint>
-<!--Camera Link
+<!--Camera Link-->
 <link name="camera">
     <collision>
@@ -133,5 +133,4 @@
         <box size="${cameraSize} ${cameraSize} ${cameraSize}"/>
       </geometry>
-      <material name="green"/>
     </visual>
     <inertial>
@@ -148,5 +147,4 @@
     <child link="camera"/>
   </joint>
--->
     <joint name="hokuyo_joint" type="fixed">
     <axis xyz="0 1 0" />

Commit message: Added Depth Camera sensor (disabled due to heating issues)

File: urdf/roomba/slambot.gazebo.xacro (robot description, xacro)
@@ -77,4 +77,31 @@
     </sensor>
   </gazebo>
+<!--Depth Camera Plugin
+  <gazebo reference="depth_cam_link">
+    <sensor type="depth" name="depth_cam">
+      <pose>0.2 0 0.055 0 0 0</pose>
+      <visualize>false</visualize>
+      <update_rate>30.0</update_rate>
+      <always_on>true</always_on>
+      <camera name="head">
+        <horizontal_fov>1.089</horizontal_fov>
+        <image>
+          <width>640</width>
+          <height>480</height>
+          <format>R8G8B8</format>
+        </image>
+        <clip>
+          <near>0.02</near>
+          <far>300</far>
+        </clip>
+      </camera>
+      <plugin name="camera_controller" filename="libgazebo_ros_camera.so">
+        <camera_name>slambot/depth_cam</camera_name>
+        <frame_name>depth_camera</frame_name>
+        <hack_baseline>0.07</hack_baseline>
+        <min_depth>0.001</min_depth>
+      </plugin>
+    </sensor>
+  </gazebo> -->
 <!-- hokuyo -->
   <gazebo reference="hokuyo">

File: urdf/roomba/slambot.xacro (robot description, xacro)
@@ -141,4 +141,31 @@
     </inertial>
   </link>
+  <joint name="depth_camera_joint" type="fixed">
+    <axis xyz="0 1 0" />
+    <origin xyz="0.2 0.1 0" rpy="0 0 0"/>
+    <parent link="chassis"/>
+    <child link="depth_cam_link"/>
+  </joint>
+<!--Depth Camera Link-->
+<link name="depth_cam_link">
+    <collision>
+      <origin xyz="0 0 0" rpy="0 0 0"/>
+      <geometry>
+        <box size="${cameraSize} ${cameraSize} ${cameraSize}"/>
+      </geometry>
+    </collision>
+    <visual>
+      <origin xyz="0 0 0" rpy="0 0 0"/>
+      <geometry>
+        <box size="${cameraSize} ${cameraSize} ${cameraSize}"/>
+      </geometry>
+    </visual>
+    <inertial>
+      <mass value="${cameraMass}" />
+      <origin xyz="0 0 0" rpy="0 0 0"/>
+      <box_inertia m="${cameraMass}" x="${cameraSize}" y="${cameraSize}" z="${cameraSize}" />
+      <inertia ixx="1e-6" ixy="0" ixz="0" iyy="1e-6" iyz="0" izz="1e-6" />
+    </inertial>
+  </link>
   <joint name="camera_joint" type="fixed">
     <axis xyz="0 1 0" />
